File: Arduino.sch (KiCad schematic (older format))
At the start: 18 parts

Commit message: Placed arduino module
Parts:
- added R49, R50, R51: R, symbol R
Connections:
- net GND: now also R50.1, R51.1
- net at R37.1: now also ARD1.21 (DIGITAL_10_MOSI); no longer ARD1.20 (DIGITAL_9_CS)
- net at ARD1.1 (5V): now also R49.2
- net at ARD1.17 (DIGITAL_6): no longer R40.1
- net at ARD1.18 (DIGITAL_7): now also R40.1; no longer R39.1
- net at ARD1.19 (DIGITAL_8): now also R39.1; no longer R38.1
- net at ARD1.2 (GND): now also R50.2
- net at R36.1: now also ARD1.22 (DIGITAL_11_MISO); no longer ARD1.21 (DIGITAL_10_MOSI)
- net at R35.1: now also ARD1.23 (DIGITAL_12_SCK); no longer ARD1.22 (DIGITAL_11_MISO)
- net at R34.1: now also ARD1.24 (DIGITAL_13); no longer ARD1.23 (DIGITAL_12_SCK)
- net at ARD1.3 (GND): now also R51.2
- new net: ARD1.20 (DIGITAL_9_CS), R38.1
- new net +5V: R49.1
Other:
- moved on the sheet: R34, R35, R36, R37, R38, R39, R40
Changed lines of the file:
@@
 Text HLabel 7900 4750 2    60   Input ~ 0
 RELAY-
-Text HLabel 5900 3850 2    60   Output ~ 0
+Text HLabel 5900 3700 2    60   Output ~ 0
 MOSI
-Text HLabel 5900 3700 2    60   Input ~ 0
+Text HLabel 5900 3550 2    60   Input ~ 0
 MISO
-Text HLabel 5900 3550 2    60   Output ~ 0
+Text HLabel 5900 3400 2    60   Output ~ 0
 SCLK
-Text HLabel 5900 4550 2    60   Output ~ 0
+Text HLabel 5900 4400 2    60   Output ~ 0
 DAC_CS_N
-Text HLabel 5900 4150 2    60   Output ~ 0
+Text HLabel 5900 4000 2    60   Output ~ 0
 LED_EN_PWM
 Text HLabel 1700 5150 0    60   Input ~ 0
@@
 L R R34
 U 1 1 52F1B473
+P 5350 3400
+F 0 "R34" V 5430 3400 40  0000 C CNN
+F 1 "R" V 5357 3401 40  0000 C CNN
+F 2 "~" V 5280 3400 30  0000 C CNN
+F 3 "~" H 5350 3400 30  0000 C CNN
+	1    5350 3400
+	0    -1   -1   0
+$EndComp
+$Comp
+L R R35
+U 1 1 52F1B480
 P 5350 3550
-F 0 "R34" V 5430 3550 40  0000 C CNN
+F 0 "R35" V 5430 3550 40  0000 C CNN
 F 1 "R" V 5357 3551 40  0000 C CNN
 F 2 "~" V 5280 3550 30  0000 C CNN
@@
 $EndComp
 $Comp
-L R R35
-U 1 1 52F1B480
+L R R36
+U 1 1 52F1B486
 P 5350 3700
-F 0 "R35" V 5430 3700 40  0000 C CNN
+F 0 "R36" V 5430 3700 40  0000 C CNN
 F 1 "R" V 5357 3701 40  0000 C CNN
 F 2 "~" V 5280 3700 30  0000 C CNN
@@
 $EndComp
 $Comp
-L R R36
-U 1 1 52F1B486
-P 5350 3850
-F 0 "R36" V 5430 3850 40  0000 C CNN
-F 1 "R" V 5357 3851 40  0000 C CNN
-F 2 "~" V 5280 3850 30  0000 C CNN
-F 3 "~" H 5350 3850 30  0000 C CNN
-	1    5350 3850
-	0    -1   -1   0
-$EndComp
-$Comp
 L R R40
 U 1 1 52F1B48C
-P 5350 4550
-F 0 "R40" V 5430 4550 40  0000 C CNN
-F 1 "R" V 5357 4551 40  0000 C CNN
-F 2 "~" V 5280 4550 30  0000 C CNN
-F 3 "~" H 5350 4550 30  0000 C CNN
-	1    5350 4550
-	0    -1   -1   0
-$EndComp
+P 5350 4400
+F 0 "R40" V 5430 4400 40  0000 C CNN
+F 1 "R" V 5357 4401 40  0000 C CNN
+F 2 "~" V 5280 4400 30  0000 C CNN
+F 3 "~" H 5350 4400 30  0000 C CNN
+	1    5350 4400
+	0    -1   -1   0
+$EndComp
+Wire Wire Line
+	4800 3400 5100 3400
 Wire Wire Line
 	4800 3550 5100 3550
@@
 	4800 3700 5100 3700
 Wire Wire Line
-	4800 3850 5100 3850
-Wire Wire Line
-	4800 4550 5100 4550
+	4800 4400 5100 4400
+Wire Wire Line
+	5600 3400 5900 3400
 Wire Wire Line
 	5600 3550 5900 3550
@@
 	5600 3700 5900 3700
 Wire Wire Line
-	5600 3850 5900 3850
-Wire Wire Line
-	5600 4550 5900 4550
+	5600 4400 5900 4400
 $Comp
 L R R42
@@
 $EndComp
 $Comp
-L GND #PWR60
+L GND #PWR059
 U 1 1 52F1B529
 P 7000 5050
-F 0 "#PWR60" H 7000 5050 30  0001 C CNN
+F 0 "#PWR059" H 7000 5050 30  0001 C CNN
 F 1 "GND" H 7000 4980 30  0001 C CNN
 F 2 "" H 7000 5050 60  0000 C CNN
@@
 L R R38
 U 1 1 52F1B568
+P 5350 4000
+F 0 "R38" V 5430 4000 40  0000 C CNN
+F 1 "R" V 5357 4001 40  0000 C CNN
+F 2 "~" V 5280 4000 30  0000 C CNN
+F 3 "~" H 5350 4000 30  0000 C CNN
+	1    5350 4000
+	0    -1   -1   0
+$EndComp
+Wire Wire Line
+	4800 4000 5100 4000
+Wire Wire Line
+	5600 4000 5900 4000
+$Comp
+L R R39
+U 1 1 52F27389
 P 5350 4150
-F 0 "R38" V 5430 4150 40  0000 C CNN
+F 0 "R39" V 5430 4150 40  0000 C CNN
 F 1 "R" V 5357 4151 40  0000 C CNN
 F 2 "~" V 5280 4150 30  0000 C CNN
@@
 Wire Wire Line
 	4800 4150 5100 4150
+Text HLabel 5900 4150 2    60   Output ~ 0
+ADC_CS_N
 Wire Wire Line
 	5600 4150 5900 4150
-$Comp
-L R R39
-U 1 1 52F27389
-P 5350 4400
-F 0 "R39" V 5430 4400 40  0000 C CNN
-F 1 "R" V 5357 4401 40  0000 C CNN
-F 2 "~" V 5280 4400 30  0000 C CNN
-F 3 "~" H 5350 4400 30  0000 C CNN
-	1    5350 4400
-	0    -1   -1   0
-$EndComp
-Wire Wire Line
-	4800 4400 5100 4400
-Text HLabel 5900 4400 2    60   Output ~ 0
-ADC_CS_N
-Wire Wire Line
-	5600 4400 5900 4400
 $Comp
 L R R37
 U 1 1 52F170F5
-P 5350 4000
-F 0 "R37" V 5430 4000 40  0000 C CNN
-F 1 "R" V 5357 4001 40  0000 C CNN
-F 2 "~" V 5280 4000 30  0000 C CNN
-F 3 "~" H 5350 4000 30  0000 C CNN
-	1    5350 4000
-	0    -1   -1   0
-$EndComp
-Wire Wire Line
-	4800 4000 5100 4000
-Wire Wire Line
-	5600 4000 5900 4000
-Text HLabel 5900 4000 2    60   Output ~ 0
+P 5350 3850
+F 0 "R37" V 5430 3850 40  0000 C CNN
+F 1 "R" V 5357 3851 40  0000 C CNN
+F 2 "~" V 5280 3850 30  0000 C CNN
+F 3 "~" H 5350 3850 30  0000 C CNN
+	1    5350 3850
+	0    -1   -1   0
+$EndComp
+Wire Wire Line
+	4800 3850 5100 3850
+Wire Wire Line
+	5600 3850 5900 3850
+Text HLabel 5900 3850 2    60   Output ~ 0
 FAN_PWM
 Text HLabel 5900 5450 2    60   Output ~ 0
@@
 	2500 4450 2700 4450
 $Comp
-L +12P #PWR59
+L +12P #PWR060
 U 1 1 52F1943B
 P 1700 4450
-F 0 "#PWR59" H 1700 4420 30  0001 C CNN
+F 0 "#PWR060" H 1700 4420 30  0001 C CNN
 F 1 "+12P" H 1700 4550 30  0000 C CNN
 F 2 "" H 1700 4450 60  0000 C CNN
@@
 Wire Wire Line
 	5600 4700 5900 4700
+$Comp
+L R R51
+U 1 1 5304B361
+P 2250 4300
+F 0 "R51" V 2330 4300 40  0000 C CNN
+F 1 "R" V 2257 4301 40  0000 C CNN
+F 2 "" V 2180 4300 30  0000 C CNN
+F 3 "" H 2250 4300 30  0000 C CNN
+	1    2250 4300
+	0    -1   -1   0
+$EndComp
+$Comp
+L R R50
+U 1 1 5304B373
+P 2250 4150
+F 0 "R50" V 2330 4150 40  0000 C CNN
+F 1 "R" V 2257 4151 40  0000 C CNN
+F 2 "" V 2180 4150 30  0000 C CNN
+F 3 "" H 2250 4150 30  0000 C CNN
+	1    2250 4150
+	0    -1   -1   0
+$EndComp
+$Comp
+L R R49
+U 1 1 5304B37E
+P 2250 4000
+F 0 "R49" V 2330 4000 40  0000 C CNN
+F 1 "R" V 2257 4001 40  0000 C CNN
+F 2 "" V 2180 4000 30  0000 C CNN
+F 3 "" H 2250 4000 30  0000 C CNN
+	1    2250 4000
+	0    -1   -1   0
+$EndComp
+Wire Wire Line
+	2000 4150 1050 4150
+Wire Wire Line
+	1050 4150 1050 4250
+$Comp
+L GND #PWR061
+U 1 1 5304B3B2
+P 1050 4250
+F 0 "#PWR061" H 1050 4250 30  0001 C CNN
+F 1 "GND" H 1050 4180 30  0001 C CNN
+F 2 "" H 1050 4250 60  0000 C CNN
+F 3 "" H 1050 4250 60  0000 C CNN
+	1    1050 4250
+	1    0    0    -1
+$EndComp
+Wire Wire Line
+	2000 4300 1850 4300
+Wire Wire Line
+	1850 4300 1850 4150
+Connection ~ 1850 4150
+Wire Wire Line
+	2000 4000 1200 4000
+Wire Wire Line
+	1200 4000 1200 3700
+$Comp
+L +5V #PWR062
+U 1 1 5304B41A
+P 1200 3700
+F 0 "#PWR062" H 1200 3790 20  0001 C CNN
+F 1 "+5V" H 1200 3790 30  0000 C CNN
+F 2 "" H 1200 3700 60  0000 C CNN
+F 3 "" H 1200 3700 60  0000 C CNN
+	1    1200 3700
+	1    0    0    -1
+$EndComp
+Wire Wire Line
+	2500 4000 2700 4000
+Wire Wire Line
+	2500 4150 2700 4150
+Wire Wire Line
+	2500 4300 2700 4300
 $EndSCHEMATC

Commit message: more changes?
Parts:
- added R52, R53: R, symbol R
Connections:
- net at ARD1.13 (DIGITAL_2): now also R53.1
- net at ARD1.14 (DIGITAL_3): now also R52.1
- net ADC_CS_N renamed ~ADC_CS
- net DAC_CS_N renamed ~DAC_CS
- new net ~LDAC: R52.2
- new net ~SHDN: R53.2
Other:
- moved on the sheet: R33
Changed lines of the file:
@@
 SCLK
 Text HLabel 5900 4400 2    60   Output ~ 0
-DAC_CS_N
+~DAC_CS
 Text HLabel 5900 4000 2    60   Output ~ 0
 LED_EN_PWM
@@
 L R R33
 U 1 1 52F1A3E5
-P 5300 5300
-F 0 "R33" V 5380 5300 40  0000 C CNN
-F 1 "R" V 5307 5301 40  0000 C CNN
-F 2 "~" V 5230 5300 30  0000 C CNN
-F 3 "~" H 5300 5300 30  0000 C CNN
-	1    5300 5300
-	0    -1   -1   0
-$EndComp
-Wire Wire Line
-	4800 5300 5050 5300
-Wire Wire Line
-	5550 5300 5900 5300
+P 5350 5300
+F 0 "R33" V 5430 5300 40  0000 C CNN
+F 1 "R" V 5357 5301 40  0000 C CNN
+F 2 "~" V 5280 5300 30  0000 C CNN
+F 3 "~" H 5350 5300 30  0000 C CNN
+	1    5350 5300
+	0    -1   -1   0
+$EndComp
+Wire Wire Line
+	4800 5300 5100 5300
+Wire Wire Line
+	5600 5300 5900 5300
 $Comp
 L R R32
@@
 $EndComp
 $Comp
-L GND #PWR059
+L GND #PWR062
 U 1 1 52F1B529
 P 7000 5050
-F 0 "#PWR059" H 7000 5050 30  0001 C CNN
+F 0 "#PWR062" H 7000 5050 30  0001 C CNN
 F 1 "GND" H 7000 4980 30  0001 C CNN
 F 2 "" H 7000 5050 60  0000 C CNN
@@
 	4800 4150 5100 4150
 Text HLabel 5900 4150 2    60   Output ~ 0
-ADC_CS_N
+~ADC_CS
 Wire Wire Line
 	5600 4150 5900 4150
@@
 	2500 4450 2700 4450
 $Comp
-L +12P #PWR060
+L +12P #PWR063
 U 1 1 52F1943B
 P 1700 4450
-F 0 "#PWR060" H 1700 4420 30  0001 C CNN
+F 0 "#PWR063" H 1700 4420 30  0001 C CNN
 F 1 "+12P" H 1700 4550 30  0000 C CNN
 F 2 "" H 1700 4450 60  0000 C CNN
@@
 $EndComp
 Wire Wire Line
-	2000 4150 1050 4150
+	1050 4150 2000 4150
 Wire Wire Line
 	1050 4150 1050 4250
 $Comp
-L GND #PWR061
+L GND #PWR064
 U 1 1 5304B3B2
 P 1050 4250
-F 0 "#PWR061" H 1050 4250 30  0001 C CNN
+F 0 "#PWR064" H 1050 4250 30  0001 C CNN
 F 1 "GND" H 1050 4180 30  0001 C CNN
 F 2 "" H 1050 4250 60  0000 C CNN
@@
 	1200 4000 1200 3700
 $Comp
-L +5V #PWR062
+L +5V #PWR065
 U 1 1 5304B41A
 P 1200 3700
-F 0 "#PWR062" H 1200 3790 20  0001 C CNN
+F 0 "#PWR065" H 1200 3790 20  0001 C CNN
 F 1 "+5V" H 1200 3790 30  0000 C CNN
 F 2 "" H 1200 3700 60  0000 C CNN
@@
 Wire Wire Line
 	2500 4300 2700 4300
+Text HLabel 5900 5000 2    60   Input ~ 0
+~LDAC
+Text HLabel 5900 5150 2    60   Output ~ 0
+~SHDN
+$Comp
+L R R52
+U 1 1 5305164B
+P 5350 5000
+F 0 "R52" V 5430 5000 40  0000 C CNN
+F 1 "R" V 5357 5001 40  0000 C CNN
+F 2 "" V 5280 5000 30  0000 C CNN
+F 3 "" H 5350 5000 30  0000 C CNN
+	1    5350 5000
+	0    -1   -1   0
+$EndComp
+$Comp
+L R R53
+U 1 1 5305165F
+P 5350 5150
+F 0 "R53" V 5430 5150 40  0000 C CNN
+F 1 "R" V 5357 5151 40  0000 C CNN
+F 2 "" V 5280 5150 30  0000 C CNN
+F 3 "" H 5350 5150 30  0000 C CNN
+	1    5350 5150
+	0    -1   -1   0
+$EndComp
+Wire Wire Line
+	4800 5000 5100 5000
+Wire Wire Line
+	5600 5000 5900 5000
+Wire Wire Line
+	4800 5150 5100 5150
+Wire Wire Line
+	5600 5150 5900 5150
 $EndSCHEMATC
