File: Power.sch (KiCad schematic (older format))
At the start: 11 parts, among them P1 24 Pin MiniFit Jr, SW1 SWITCH_INV

Commit message: associated power module
Parts:
- added C13: C, ~, symbol C
- added L4: CM322522-220KL, ~, symbol INDUCTOR
- L1, L2: value INDUCTOR -> CM322522-220KL; MFG Part Number (none) -> CM322522-220KL
- SW1: value SWITCH_INV -> Power Switch; MFG Name (none) -> C & K Components; MFG Part Number (none) -> OS102011MA1QN1
- TH1: MFG Part Number (none) -> MINISMDC050F-2 MINISMDC050F-2
- TH2, TH3, TH4: MFG Part Number (none) -> MINISMDC050F-2
Connections:
- net labels added: +5P
- wire segments 38 -> 44
Changed lines of the file:
@@
 $EndComp
 Wire Wire Line
-	2150 2950 1600 2950
+	1600 2950 2150 2950
 Wire Wire Line
 	1600 2950 1600 3150
 $Comp
-L GND #PWR018
+L GND #PWR18
 U 1 1 52EFD186
 P 1600 3150
-F 0 "#PWR018" H 1600 3150 30  0001 C CNN
+F 0 "#PWR18" H 1600 3150 30  0001 C CNN
 F 1 "GND" H 1600 3080 30  0001 C CNN
 F 2 "" H 1600 3150 60  0000 C CNN
@@
 $EndComp
 $Comp
-L +3.3V #PWR019
+L +3.3V #PWR20
 U 1 1 52EFD19A
 P 3900 2450
-F 0 "#PWR019" H 3900 2410 30  0001 C CNN
+F 0 "#PWR20" H 3900 2410 30  0001 C CNN
 F 1 "+3.3V" H 3900 2560 30  0000 C CNN
 F 2 "" H 3900 2450 60  0000 C CNN
@@
 $EndComp
 $Comp
-L +5V #PWR020
+L +5V #PWR21
 U 1 1 52EFD1B0
 P 4700 2450
-F 0 "#PWR020" H 4700 2540 20  0001 C CNN
+F 0 "#PWR21" H 4700 2540 20  0001 C CNN
 F 1 "+5V" H 4700 2540 30  0000 C CNN
 F 2 "" H 4700 2450 60  0000 C CNN
@@
 	5500 3250 5500 2450
 $Comp
-L +12P #PWR021
+L +12P #PWR24
 U 1 1 52EFD28E
 P 5500 2450
-F 0 "#PWR021" H 5500 2420 30  0001 C CNN
+F 0 "#PWR24" H 5500 2420 30  0001 C CNN
 F 1 "+12P" H 5500 2550 30  0000 C CNN
 F 2 "" H 5500 2450 60  0000 C CNN
@@
 $EndComp
 $Comp
-L -12P #PWR022
+L -12P #PWR25
 U 1 1 52EFD366
 P 6450 2450
-F 0 "#PWR022" H 6450 2420 30  0001 C CNN
+F 0 "#PWR25" H 6450 2420 30  0001 C CNN
 F 1 "-12P" H 6450 2550 30  0000 C CNN
 F 2 "" H 6450 2450 60  0000 C CNN
@@
 P 3950 4600
 F 0 "SW1" H 3750 4750 50  0000 C CNN
-F 1 "SWITCH_INV" H 3800 4450 50  0000 C CNN
+F 1 "Power Switch" H 3800 4450 50  0000 C CNN
 F 2 "~" H 3950 4600 60  0000 C CNN
 F 3 "~" H 3950 4600 60  0000 C CNN
+F 4 "C & K Components" H 3950 4600 60  0001 C CNN "MFG Name"
+F 5 "OS102011MA1QN1" H 3950 4600 60  0001 C CNN "MFG Part Number"
 	1    3950 4600
 	1    0    0    -1
@@
 	4700 4700 4700 5000
 $Comp
-L GND #PWR023
+L GND #PWR22
 U 1 1 52EFD4D4
 P 4700 5000
-F 0 "#PWR023" H 4700 5000 30  0001 C CNN
+F 0 "#PWR22" H 4700 5000 30  0001 C CNN
 F 1 "GND" H 4700 4930 30  0001 C CNN
 F 2 "" H 4700 5000 60  0000 C CNN
@@
 	5350 4500 5350 4200
 $Comp
-L +3.3V #PWR024
+L +3.3V #PWR23
 U 1 1 52EFD557
 P 5350 4200
-F 0 "#PWR024" H 5350 4160 30  0001 C CNN
+F 0 "#PWR23" H 5350 4160 30  0001 C CNN
 F 1 "+3.3V" H 5350 4310 30  0000 C CNN
 F 2 "" H 5350 4200 60  0000 C CNN
@@
 $EndComp
 $Comp
-L +12P #PWR025
+L +12P #PWR26
 U 1 1 52EFD66E
 P 7400 3750
-F 0 "#PWR025" H 7400 3720 30  0001 C CNN
+F 0 "#PWR26" H 7400 3720 30  0001 C CNN
 F 1 "+12P" H 7400 3850 30  0000 C CNN
 F 2 "" H 7400 3750 60  0000 C CNN
@@
 $EndComp
 $Comp
-L -12P #PWR026
+L -12P #PWR28
 U 1 1 52EFD674
 P 7400 5150
-F 0 "#PWR026" H 7400 5120 30  0001 C CNN
+F 0 "#PWR28" H 7400 5120 30  0001 C CNN
 F 1 "-12P" H 7400 5250 30  0000 C CNN
 F 2 "" H 7400 5150 60  0000 C CNN
@@
 $EndComp
 $Comp
-L GND #PWR027
+L GND #PWR27
 U 1 1 52EFD67A
 P 7400 4500
-F 0 "#PWR027" H 7400 4500 30  0001 C CNN
+F 0 "#PWR27" H 7400 4500 30  0001 C CNN
 F 1 "GND" H 7400 4430 30  0001 C CNN
 F 2 "" H 7400 4500 60  0000 C CNN
@@
 P 8050 3900
 F 0 "L2" V 8000 3900 40  0000 C CNN
-F 1 "INDUCTOR" V 8150 3900 40  0000 C CNN
+F 1 "CM322522-220KL" V 8150 3900 40  0000 C CNN
 F 2 "~" H 8050 3900 60  0000 C CNN
 F 3 "~" H 8050 3900 60  0000 C CNN
+F 4 "CM322522-220KL" H 8050 3900 60  0001 C CNN "MFG Part Number"
 	1    8050 3900
 	0    -1   -1   0
@@
 P 8000 5100
 F 0 "L1" V 7950 5100 40  0000 C CNN
-F 1 "INDUCTOR" V 8100 5100 40  0000 C CNN
+F 1 "CM322522-220KL" V 8100 5100 40  0000 C CNN
 F 2 "~" H 8000 5100 60  0000 C CNN
 F 3 "~" H 8000 5100 60  0000 C CNN
+F 4 "CM322522-220KL" H 8000 5100 60  0001 C CNN "MFG Part Number"
 	1    8000 5100
 	0    -1   -1   0
@@
 Connection ~ 8700 4400
 $Comp
-L +12V #PWR028
+L +12V #PWR31
 U 1 1 52EFD773
 P 9150 3750
-F 0 "#PWR028" H 9150 3700 20  0001 C CNN
+F 0 "#PWR31" H 9150 3700 20  0001 C CNN
 F 1 "+12V" H 9150 3850 30  0000 C CNN
 F 2 "" H 9150 3750 60  0000 C CNN
@@
 	7400 5100 7700 5100
 $Comp
-L -12V #PWR029
+L -12V #PWR32
 U 1 1 52EFD7D2
 P 9150 5250
-F 0 "#PWR029" H 9150 5380 20  0001 C CNN
+F 0 "#PWR32" H 9150 5380 20  0001 C CNN
 F 1 "-12V" H 9150 5350 30  0000 C CNN
 F 2 "" H 9150 5250 60  0000 C CNN
@@
 Connection ~ 3200 3250
 $Comp
-L +12C #PWR030
+L +12C #PWR19
 U 1 1 52F156A2
 P 3200 2400
-F 0 "#PWR030" H 3200 2370 30  0001 C CNN
+F 0 "#PWR19" H 3200 2370 30  0001 C CNN
 F 1 "+12C" H 3200 2510 40  0000 C CNN
 F 2 "" H 3200 2400 60  0000 C CNN
@@
 F 2 "~" H 3500 2850 60  0000 C CNN
 F 3 "~" H 3500 2850 60  0000 C CNN
+F 4 "MINISMDC050F-2MINISMDC050F-2" H 3500 2850 60  0001 C CNN "MFG Part Number"
 	1    3500 2850
 	0    -1   -1   0
@@
 F 2 "~" H 4300 3050 60  0000 C CNN
 F 3 "~" H 4300 3050 60  0000 C CNN
+F 4 "MINISMDC050F-2" H 4300 3050 60  0001 C CNN "MFG Part Number"
 	1    4300 3050
 	0    -1   -1   0
@@
 F 2 "~" H 5050 3250 60  0000 C CNN
 F 3 "~" H 5050 3250 60  0000 C CNN
+F 4 "MINISMDC050F-2" H 5050 3250 60  0001 C CNN "MFG Part Number"
 	1    5050 3250
 	0    -1   -1   0
@@
 F 2 "~" H 5950 3450 60  0000 C CNN
 F 3 "~" H 5950 3450 60  0000 C CNN
+F 4 "MINISMDC050F-2" H 5950 3450 60  0001 C CNN "MFG Part Number"
 	1    5950 3450
 	0    -1   -1   0
 $EndComp
+$Comp
+L GND #PWR30
+U 1 1 530781BE
+P 8700 2900
+F 0 "#PWR30" H 8700 2900 30  0001 C CNN
+F 1 "GND" H 8700 2830 30  0001 C CNN
+F 2 "" H 8700 2900 60  0000 C CNN
+F 3 "" H 8700 2900 60  0000 C CNN
+	1    8700 2900
+	1    0    0    -1
+$EndComp
+$Comp
+L C C13
+U 1 1 530781C9
+P 8700 2550
+F 0 "C13" H 8700 2650 40  0000 L CNN
+F 1 "C" H 8706 2465 40  0000 L CNN
+F 2 "~" H 8738 2400 30  0000 C CNN
+F 3 "~" H 8700 2550 60  0000 C CNN
+	1    8700 2550
+	1    0    0    -1
+$EndComp
+$Comp
+L INDUCTOR L4
+U 1 1 530781D5
+P 8150 2150
+F 0 "L4" V 8100 2150 40  0000 C CNN
+F 1 "CM322522-220KL" V 8250 2150 40  0000 C CNN
+F 2 "~" H 8150 2150 60  0000 C CNN
+F 3 "~" H 8150 2150 60  0000 C CNN
+F 4 "CM322522-220KL" H 8150 2150 60  0001 C CNN "MFG Part Number"
+	1    8150 2150
+	0    -1   -1   0
+$EndComp
+$Comp
+L +5P #PWR29
+U 1 1 530781E3
+P 7450 1950
+F 0 "#PWR29" H 7450 2080 20  0001 C CNN
+F 1 "+5P" H 7450 2050 30  0000 C CNN
+F 2 "" H 7450 1950 60  0000 C CNN
+F 3 "" H 7450 1950 60  0000 C CNN
+	1    7450 1950
+	1    0    0    -1
+$EndComp
+$Comp
+L +5V #PWR33
+U 1 1 530781F7
+P 9250 1900
+F 0 "#PWR33" H 9250 1990 20  0001 C CNN
+F 1 "+5V" H 9250 1990 30  0000 C CNN
+F 2 "" H 9250 1900 60  0000 C CNN
+F 3 "" H 9250 1900 60  0000 C CNN
+	1    9250 1900
+	1    0    0    -1
+$EndComp
+Wire Wire Line
+	7450 1950 7450 2150
+Wire Wire Line
+	7450 2150 7850 2150
+Wire Wire Line
+	8450 2150 9250 2150
+Wire Wire Line
+	9250 2150 9250 1900
+Wire Wire Line
+	8700 2350 8700 2150
+Connection ~ 8700 2150
+Wire Wire Line
+	8700 2750 8700 2900
 $EndSCHEMATC
